Commit message: Add xArm6 workcells and dual Ouster sensing
Pin the manufacturer robot description and cam_wip Ouster sources, including recursive dependencies. Share SDF geometry between Gazebo, MoveIt collision checking, and scene markers.

Run Gazebo headless with Foxglove Bridge, named-pose commands, and optional dual-cloud occupancy mapping. Correct the cam_wip decoder frames and keep desktop mesh URIs portable.

Validate scene composition, collision-aware execution, WebSocket publishing and assets, and geometric cloud registration.

File: src/arm_description/urdf/arm.urdf.xacro (robot description, xacro)
@@ -3,4 +3,7 @@
   <xacro:arg name="hardware" default="mock"/>
   <xacro:arg name="controllers_file" default=""/>
+  <xacro:arg name="mount_xyz" default="0 0 0"/>
+  <xacro:arg name="mount_rpy" default="0 0 0"/>
+  <xacro:include filename="$(find arm_description)/urdf/materials.xacro"/>
   <xacro:property name="hardware" value="$(arg hardware)"/>
   <material name="blue"><color rgba="0.12 0.38 0.75 1"/></material>
@@ -13,5 +16,5 @@
     <inertial><origin xyz="0 0 0.05"/><mass value="3"/><inertia ixx="0.0125" ixy="0" ixz="0" iyy="0.0125" iyz="0" izz="0.02"/></inertial>
   </link>
-  <joint name="world_joint" type="fixed"><parent link="world"/><child link="base_link"/></joint>
+  <joint name="world_joint" type="fixed"><parent link="world"/><child link="base_link"/><origin xyz="$(arg mount_xyz)" rpy="$(arg mount_rpy)"/></joint>
   <xacro:macro name="arm_segment" params="index parent offset length radius mass axis color">
     <link name="link_${index}">
@@ -37,4 +40,11 @@
   <xacro:arm_segment index="5" parent="link_4" offset="0.10" length="0.08" radius="0.025" mass="0.2" axis="0 1 0" color="blue"/>
   <xacro:arm_segment index="6" parent="link_5" offset="0.08" length="0.08" radius="0.022" mass="0.15" axis="0 0 1" color="silver"/>
+  <xacro:gazebo_surface link="base_link" color="0.15 0.17 0.20 1"/>
+  <xacro:gazebo_surface link="link_1" color="0.65 0.68 0.72 1" metalness="0.6"/>
+  <xacro:gazebo_surface link="link_2" color="0.12 0.38 0.75 1"/>
+  <xacro:gazebo_surface link="link_3" color="0.12 0.38 0.75 1"/>
+  <xacro:gazebo_surface link="link_4" color="0.65 0.68 0.72 1" metalness="0.6"/>
+  <xacro:gazebo_surface link="link_5" color="0.12 0.38 0.75 1"/>
+  <xacro:gazebo_surface link="link_6" color="0.65 0.68 0.72 1" metalness="0.6"/>
   <link name="tool0"/>
   <joint name="tool_joint" type="fixed"><parent link="link_6"/><child link="tool0"/><origin xyz="0 0 0.08"/></joint>
