Commit message: Run Ousters at 10 Hz in real time; add xArm Gripper, cameras, and picks
Simulation performance (measured in Docker on a 4-vCPU VM; RTF 0.99-1.01
with both Ousters at 10 Hz wall and sim time, from 0.72 and lossy clouds):

- Cyclone DDS: 64 KB fragments (docker/cyclonedds.xml) and reliable lidar
  packets and clouds. A 3.1 MB cloud in 1.3 KB fragments overran Docker
  Desktop's ~208 KB socket buffers, so best-effort subscribers lost most
  scans.
- arm_bringup::RealtimePacer: paces steps against an absolute wall-clock
  schedule and repays late wake-ups (worlds set real_time_factor 0);
  gz-sim's own throttle drops that time and held the container near 0.8.
- gz_relay: republishes Gazebo's 1 kHz clock as /clock at 200 Hz and part
  poses from dynamic_pose/info, instead of per-step ROS wake-ups and
  per-part PosePublisher systems. Altimeter system dropped.
- Bullet Featherstone physics: enforces the gripper's mimic joints natively;
  servoing them through gz_ros2_control under DART cost 18% of real time.
- Ousters default to 10 Hz; OMP_WAIT_POLICY=PASSIVE; the gz_sensors_ouster
  submodule moves to the row-balanced CPU raycaster (perf/cpu-raycast-m1).
- The workcell UI asks MoveIt for the hand pose instead of decoding /tf, and
  runs without use_sim_time in Gazebo (a Python /clock subscriber costs ~9%
  of a core).

Manipulation and sensing:

- UFACTORY xArm Gripper (xarm_gripper.xacro): manufacturer kinematics and
  meshes, primitive collisions, URDF mimic linkage, drive_joint at the rated
  grip force, parallel_gripper_action_controller, MoveIt group with open
  (85 mm) and close states.
- RealSense cameras (cameras.xacro): a D435i on UFACTORY's wrist stand and
  an overhead D455, as separate color and depth sensors with realsense-ros
  topics, bridged lazily so unwatched cameras cost nothing.
- Movable parts: single-link SDF models are mirrored into MoveIt from
  Gazebo's poses. /motion/command pick_cube and pick_cylinder run a top-down
  pick and place through MoveIt (IK-filtered grasp yaws, Cartesian descent
  and lift, attached collision objects). After the gripper closes and stalls
  on a part, arm_bringup::GraspWeld welds it to the hand until release
  (weld_grasps:=false holds by friction only), since Bullet's point contacts
  let a held cylinder tip and fall.
- Checks: check_rates.py (rates, scan completeness, RTF), check_pick.py
  (part placement in Gazebo), make rates-check / pick-check, a pick in the
  Gazebo smoke test, gripper checks in check_stack, and pick geometry unit
  tests. Lichtblick layout gains camera panels and pick/gripper buttons.

Co-Authored-By: Claude Opus 5.5 <noreply@anthropic.com>
Claude-Session: https://claude.ai/code/session_015jsjLXS2XXuwPhcf7UDz3m

File: src/arm_description/urdf/world_sensors.urdf.xacro (robot description, xacro)
@@ -2,17 +2,29 @@
 <robot xmlns:xacro="http://www.ros.org/wiki/xacro" name="workcell_sensors">
   <xacro:arg name="metadata_path" default=""/>
+  <xacro:arg name="ousters" default="true"/>
   <xacro:arg name="front_xyz" default="1.35 -1.1 1.85"/>
   <xacro:arg name="front_rpy" default="0 0.5 2.5"/>
   <xacro:arg name="rear_xyz" default="-1.25 1.15 2.15"/>
   <xacro:arg name="rear_rpy" default="0 0.65 -0.7"/>
-  <xacro:arg name="lidar_hz" default="3.0"/>
+  <xacro:arg name="lidar_hz" default="10.0"/>
+  <xacro:arg name="overhead_camera" default="false"/>
+  <xacro:arg name="overhead_xyz" default="0 0 2.1"/>
+  <xacro:arg name="overhead_rpy" default="0 1.5708 1.5708"/>
+  <xacro:arg name="overhead_hz" default="10.0"/>
   <link name="sensor_rig">
     <inertial><mass value="0.1"/><inertia ixx="0.001" ixy="0" ixz="0" iyy="0.001" iyz="0" izz="0.001"/></inertial>
   </link>
-  <xacro:include filename="$(find gz_sensors_ouster)/examples/urdf/ouster_macro.xacro"/>
-  <xacro:ouster_sensor name="ouster_front" parent="sensor_rig" metadata_path="$(arg metadata_path)"
-      xyz="$(arg front_xyz)" rpy="$(arg front_rpy)" lidar_hz="$(arg lidar_hz)" ray_mode="raycast"/>
-  <xacro:ouster_sensor name="ouster_rear" parent="sensor_rig" metadata_path="$(arg metadata_path)"
-      xyz="$(arg rear_xyz)" rpy="$(arg rear_rpy)" lidar_hz="$(arg lidar_hz)" ray_mode="raycast"/>
+  <xacro:if value="$(arg ousters)">
+    <xacro:include filename="$(find gz_sensors_ouster)/examples/urdf/ouster_macro.xacro"/>
+    <xacro:ouster_sensor name="ouster_front" parent="sensor_rig" metadata_path="$(arg metadata_path)"
+        xyz="$(arg front_xyz)" rpy="$(arg front_rpy)" lidar_hz="$(arg lidar_hz)" ray_mode="raycast"/>
+    <xacro:ouster_sensor name="ouster_rear" parent="sensor_rig" metadata_path="$(arg metadata_path)"
+        xyz="$(arg rear_xyz)" rpy="$(arg rear_rpy)" lidar_hz="$(arg lidar_hz)" ray_mode="raycast"/>
+  </xacro:if>
+  <xacro:if value="$(arg overhead_camera)">
+    <xacro:include filename="$(find arm_description)/urdf/cameras.xacro"/>
+    <xacro:fixed_d455 name="overhead" parent="sensor_rig" xyz="$(arg overhead_xyz)" rpy="$(arg overhead_rpy)"
+        update_rate="$(arg overhead_hz)"/>
+  </xacro:if>
   <gazebo><static>true</static></gazebo>
 </robot>

File: src/arm_description/urdf/xarm6.urdf.xacro (robot description, xacro)
@@ -5,4 +5,9 @@
   <xacro:arg name="mount_xyz" default="0 0 0"/>
   <xacro:arg name="mount_rpy" default="0 0 0"/>
+  <!-- UFACTORY xArm Gripper on the flange, and the RealSense D435i camera
+       stand UFACTORY mounts between flange and gripper. -->
+  <xacro:arg name="gripper" default="true"/>
+  <xacro:arg name="wrist_camera" default="true"/>
+  <xacro:arg name="camera_hz" default="15.0"/>
   <xacro:property name="hardware" value="$(arg hardware)"/>
   <xacro:property name="control_plugin" value="${'gz_ros2_control/GazeboSimSystem' if hardware == 'gazebo' else 'mock_components/GenericSystem'}"/>
@@ -15,5 +20,7 @@
   <xacro:xarm_materials/>
   <xacro:include filename="$(find xarm_description)/urdf/common/common.link.xacro"/>
-  <xacro:include filename="$(find xarm_description)/urdf/xarm6/xarm6_robot_macro.xacro"/>
+  <xacro:include filename="$(find xarm_description)/urdf/xarm6/xarm6.urdf.xacro"/>
+  <xacro:include filename="$(find xarm_description)/urdf/xarm6/xarm6.transmission.xacro"/>
+  <xacro:include filename="$(find xarm_description)/urdf/xarm6/xarm6.gazebo.xacro"/>
   <link name="world"/>
   <joint name="world_joint" type="fixed">
@@ -21,8 +28,55 @@
     <origin xyz="$(arg mount_xyz)" rpy="$(arg mount_rpy)"/>
   </joint>
-  <xacro:xarm6_robot limited="true" ros2_control_plugin="${control_plugin}"
+  <!-- UFACTORY's xarm6_robot macro with limited="true", minus its ros2_control
+       block, which cannot set initial joint positions. -->
+  <xacro:property name="limits" value="${[(-pi*0.99, pi*0.99), (-2.059, 2.0944), (-pi*0.99, 0.19198),
+                                         (-pi*0.99, pi*0.99), (-1.69297, pi*0.99), (-pi*0.99, pi*0.99)]}"/>
+  <xacro:xarm6_urdf prefix=""
+      joint1_lower_limit="${limits[0][0]}" joint1_upper_limit="${limits[0][1]}"
+      joint2_lower_limit="${limits[1][0]}" joint2_upper_limit="${limits[1][1]}"
+      joint3_lower_limit="${limits[2][0]}" joint3_upper_limit="${limits[2][1]}"
+      joint4_lower_limit="${limits[3][0]}" joint4_upper_limit="${limits[3][1]}"
+      joint5_lower_limit="${limits[4][0]}" joint5_upper_limit="${limits[4][1]}"
+      joint6_lower_limit="${limits[5][0]}" joint6_upper_limit="${limits[5][1]}"
       kinematics_params_filename="$(find xarm_description)/config/kinematics/default/xarm6_default_kinematics.yaml"/>
-  <link name="link_eef"/>
+  <xacro:xarm6_transmission prefix="" hard_interface="PositionJointInterface"/>
+  <xacro:xarm6_gazebo prefix=""/>
+  <!-- Start at the SRDF's home pose. With a gripper, the all-zero pose points
+       the fingers into the bench, so home is UFACTORY's "hold-up" pose
+       (joint5 = -90 deg). Keep in step with arm_moveit_config xarm6/arm.srdf.xacro. -->
+  <xacro:property name="home" value="${[0, 0, 0, 0, -1.5708 if '$(arg gripper)' == 'true' else 0, 0]}"/>
+  <xacro:macro name="arm_joint" params="index">
+    <joint name="joint${index}">
+      <command_interface name="position">
+        <param name="min">${limits[index - 1][0]}</param><param name="max">${limits[index - 1][1]}</param>
+      </command_interface>
+      <command_interface name="velocity"><param name="min">-3.14</param><param name="max">3.14</param></command_interface>
+      <state_interface name="position"><param name="initial_value">${home[index - 1]}</param></state_interface>
+      <state_interface name="velocity"/>
+    </joint>
+  </xacro:macro>
+  <ros2_control name="XArm6System" type="system">
+    <hardware><plugin>${control_plugin}</plugin></hardware>
+    <xacro:arm_joint index="1"/><xacro:arm_joint index="2"/><xacro:arm_joint index="3"/>
+    <xacro:arm_joint index="4"/><xacro:arm_joint index="5"/><xacro:arm_joint index="6"/>
+  </ros2_control>
+  <xacro:if value="$(arg wrist_camera)">
+    <!-- link_eef becomes UFACTORY's camera stand, with the D435i frame tree. -->
+    <xacro:include filename="$(find xarm_description)/urdf/camera/realsense_d435i.urdf.xacro"/>
+    <xacro:d435i_urdf add_d435i_links="true"/>
+    <xacro:include filename="$(find arm_description)/urdf/cameras.xacro"/>
+    <xacro:if value="${hardware == 'gazebo'}">
+      <xacro:d435i_camera name="wrist" color_link="camera_color_frame" color_optical="camera_color_optical_frame"
+          depth_link="camera_depth_frame" depth_optical="camera_depth_optical_frame" update_rate="$(arg camera_hz)"/>
+    </xacro:if>
+  </xacro:if>
+  <xacro:unless value="$(arg wrist_camera)">
+    <link name="link_eef"/>
+  </xacro:unless>
   <joint name="joint_eef" type="fixed"><parent link="link6"/><child link="link_eef"/></joint>
+  <xacro:if value="$(arg gripper)">
+    <xacro:include filename="$(find arm_description)/urdf/xarm_gripper.xacro"/>
+    <xacro:xarm_gripper attach_to="link_eef" control_plugin="${control_plugin}"/>
+  </xacro:if>
   <xacro:gazebo_surface link="link_base" color="0.88 0.91 0.93 1"/>
   <xacro:gazebo_surface link="link1" color="0.88 0.91 0.93 1"/>
