Commit message: Make the RealSense cameras faster and closer to the real devices
Camera rendering, not the sim, limited the real-time factor once images
were watched: on the M1 and on a 4-vCPU VM, subscribing to all four images
held the simulation at ~0.25-0.28. Docker has no GPU, so Mesa's software
rasterizer draws every image. Measured one change at a time on the VM
(all four images subscribed):

- No shadow-casting lights (0.28 -> 0.40): every shadowed light rendered
  shadow maps per camera image.
- No MSAA on color images (-> 0.67); camera_anti_aliasing:=4 restores
  Gazebo's default.
- Overhead D455 at 15 Hz (-> 0.83): 10 Hz is not a D455 mode, and at 15 Hz
  both cameras' images render together instead of overrunning each other.
- Robot meshes reduced to within 1 mm (0.5 mm for the gripper) of
  UFACTORY's, 130k -> 53k triangles (arm_description/meshes/sim,
  scripts/simplify_meshes.py); MoveIt and physics use them too.
- Controller spawner switch/service timeouts raised to 60 s: a cold host's
  first shader compile stalled Gazebo past the 10 s call timeout.

Accuracy:

- depth/image_rect_raw is now what a D4xx and realsense-ros publish: 16UC1
  millimetres, 0 for no depth, with stereo error RMS z^2 * 0.08 /
  (focal_px * baseline). arm_bringup/realsense_depth adds it, reading
  Gazebo's depth directly and only while watched; it measured to the model
  in every range bin (scripts/check_realsense.py, make camera-check). The
  ideal depth moves to depth/image_meters as ground truth.
- The overhead D455's frames follow realsense-ros: camera_link is the depth
  imager, the color imager 59 mm away, the case centred 47.5 mm away.

Final: 0.76-0.78 with all four images (run-to-run spread up to 0.04), 1.00
with none watched; picks land within 2 mm.

The D435i IMU was evaluated and left out: under Bullet Featherstone,
Gazebo's IMU gets no link rotation rate or acceleration (the gyro read
noise while the wrist turned at 0.4 rad/s; under DART it tracked).

Co-Authored-By: Claude Opus 5.5 <noreply@anthropic.com>
Claude-Session: https://claude.ai/code/session_015jsjLXS2XXuwPhcf7UDz3m

File: src/arm_description/urdf/cameras.xacro (robot description, xacro)
@@ -1,17 +1,20 @@
 <?xml version="1.0"?>
 <!--
-  RealSense-style RGB-D cameras for gz-sim: a color camera and a depth camera
-  on their own frames and fields of view, as on the device (and as
-  realsense-ros publishes them without alignment).
+  RealSense cameras for gz-sim: a color camera and a depth camera on their own
+  frames and fields of view, as on the device (and as realsense-ros publishes
+  them without alignment).
   Gazebo topics  /camera/<name>/color/{image,camera_info}
-                 /camera/<name>/depth/{image,camera_info,points}
+                 /camera/<name>/depth/{image,camera_info,image/points}
   frame_id       the optical frame of each imager (z forward, x right, y down)
-  Separate sensors rather than one rgbd_camera: gz-sim's rgbd_camera renders
-  lit geometry black in its color image under Mesa's llvmpipe, which is what
-  renders in Docker on a Mac. Gazebo renders a sensor only while something
-  subscribes to it, and the launch bridges these topics lazily, so an
-  unwatched stream costs nothing.
+  Separate sensors rather than one rgbd_camera keep each imager's field of
+  view and position. Gazebo renders a sensor only while something subscribes
+  to it, and the launch bridges these topics lazily, so an unwatched stream
+  costs nothing. Under Docker on a Mac every image is drawn by Mesa's software
+  renderer, and 4x MSAA (Gazebo's default) multiplied each color image's cost:
+  anti-aliasing is off unless camera_anti_aliasing is set. The includer
+  declares that xacro argument.
 -->
 <robot xmlns:xacro="http://www.ros.org/wiki/xacro">
+  <xacro:property name="camera_anti_aliasing" value="$(arg camera_anti_aliasing)"/>
   <!-- link: x-forward body frame (REP 103), the direction gz-sim cameras look. -->
   <xacro:macro name="gz_camera" params="name stream type link optical_frame width height hfov
@@ -28,5 +31,6 @@
           <horizontal_fov>${hfov}</horizontal_fov>
           <image><width>${width}</width><height>${height}</height>
-            <format>${'R8G8B8' if type == 'camera' else 'R_FLOAT32'}</format></image>
+            <format>${'R8G8B8' if type == 'camera' else 'R_FLOAT32'}</format>
+            <anti_aliasing>${camera_anti_aliasing if type == 'camera' else 0}</anti_aliasing></image>
           <clip><near>${near}</near><far>${far}</far></clip>
           <xacro:if value="${noise > 0}">
@@ -40,5 +44,7 @@
   </xacro:macro>
   <!-- Intel RealSense D435i: color 640x360 at 69.4 x 42.5 deg; depth 640x360
-       at 87 x 56 deg, 0.17 m minimum depth at this resolution, 10 m range. -->
+       at 87 x 56 deg, 0.17 m minimum depth at this resolution, 10 m range.
+       15 fps is a native mode of both imagers. Depth noise is added downstream
+       (arm_bringup realsense_depth), since Gazebo's is range-independent. -->
   <xacro:macro name="d435i_camera" params="name color_link color_optical depth_link depth_optical
                                            update_rate:=15.0">
@@ -51,7 +57,8 @@
   </xacro:macro>
   <!-- Intel RealSense D455: color 640x400 at 90 x 65 deg; depth 640x360 at
-       87 x 56 deg, 0.4 m minimum depth, ~6 m useful range. -->
+       87 x 56 deg, 0.4 m minimum depth, ~6 m useful range. 15 fps is a native
+       mode of both imagers (10 is not). -->
   <xacro:macro name="d455_camera" params="name color_link color_optical depth_link depth_optical
-                                          update_rate:=10.0">
+                                          update_rate:=15.0">
     <xacro:gz_camera name="${name}" stream="color" type="camera" link="${color_link}"
         optical_frame="${color_optical}" width="640" height="400" hfov="1.5708"
@@ -61,13 +68,15 @@
         update_rate="${update_rate}" near="0.4" far="6.0" noise="0"/>
   </xacro:macro>
-  <!-- A fixed D455 with realsense-ros frame names under <name>_camera_*.
-       Color and depth share the camera_link origin here. -->
-  <xacro:macro name="fixed_d455" params="name parent xyz rpy update_rate:=10.0">
+  <!-- A fixed D455 with realsense-ros frame names under <name>_camera_*. As in
+       realsense-ros (_d455.urdf.xacro), <name>_camera_link is the depth
+       (left infrared) imager; the color imager sits 59 mm toward the right
+       infrared imager and the case centre 47.5 mm. The optical centres are at
+       the front glass, so the case sits behind them; a sensor inside the case
+       would see its inner faces. -->
+  <xacro:macro name="fixed_d455" params="name parent xyz rpy update_rate:=15.0">
     <link name="${name}_camera_link">
       <inertial><mass value="0.39"/><inertia ixx="1e-4" ixy="0" ixz="0" iyy="1e-4" iyz="0" izz="1e-4"/></inertial>
       <visual>
-        <!-- The optical centres are at the front glass, so the body sits
-             behind them; a sensor inside the body would see its inner faces. -->
-        <origin xyz="-0.0155 0 0" rpy="0 0 0"/>
+        <origin xyz="-0.0155 -0.0475 0" rpy="0 0 0"/>
         <geometry><box size="0.029 0.124 0.026"/></geometry>
         <material name="camera_dark"><color rgba="0.12 0.13 0.15 1"/></material>
@@ -78,15 +87,20 @@
       <origin xyz="${xyz}" rpy="${rpy}"/>
     </joint>
-    <xacro:macro name="optical" params="stream">
+    <xacro:macro name="imager" params="stream y">
+      <link name="${name}_camera_${stream}_frame"/>
+      <joint name="${name}_camera_${stream}_joint" type="fixed">
+        <parent link="${name}_camera_link"/><child link="${name}_camera_${stream}_frame"/>
+        <origin xyz="0 ${y} 0" rpy="0 0 0"/>
+      </joint>
       <link name="${name}_camera_${stream}_optical_frame"/>
       <joint name="${name}_camera_${stream}_optical_joint" type="fixed">
-        <parent link="${name}_camera_link"/><child link="${name}_camera_${stream}_optical_frame"/>
+        <parent link="${name}_camera_${stream}_frame"/><child link="${name}_camera_${stream}_optical_frame"/>
         <origin xyz="0 0 0" rpy="${-pi/2} 0 ${-pi/2}"/>
       </joint>
     </xacro:macro>
-    <xacro:optical stream="color"/>
-    <xacro:optical stream="depth"/>
-    <xacro:d455_camera name="${name}" color_link="${name}_camera_link"
-        color_optical="${name}_camera_color_optical_frame" depth_link="${name}_camera_link"
+    <xacro:imager stream="depth" y="0"/>
+    <xacro:imager stream="color" y="-0.059"/>
+    <xacro:d455_camera name="${name}" color_link="${name}_camera_color_frame"
+        color_optical="${name}_camera_color_optical_frame" depth_link="${name}_camera_depth_frame"
         depth_optical="${name}_camera_depth_optical_frame" update_rate="${update_rate}"/>
   </xacro:macro>

File: src/arm_description/urdf/world_sensors.urdf.xacro (robot description, xacro)
@@ -11,5 +11,6 @@
   <xacro:arg name="overhead_xyz" default="0 0 2.1"/>
   <xacro:arg name="overhead_rpy" default="0 1.5708 1.5708"/>
-  <xacro:arg name="overhead_hz" default="10.0"/>
+  <xacro:arg name="overhead_hz" default="15.0"/>
+  <xacro:arg name="camera_anti_aliasing" default="0"/>
   <link name="sensor_rig">
     <inertial><mass value="0.1"/><inertia ixx="0.001" ixy="0" ixz="0" iyy="0.001" iyz="0" izz="0.001"/></inertial>

File: src/arm_description/urdf/xarm6.urdf.xacro (robot description, xacro)
@@ -10,4 +10,5 @@
   <xacro:arg name="wrist_camera" default="true"/>
   <xacro:arg name="camera_hz" default="15.0"/>
+  <xacro:arg name="camera_anti_aliasing" default="0"/>
   <xacro:property name="hardware" value="$(arg hardware)"/>
   <xacro:property name="control_plugin" value="${'gz_ros2_control/GazeboSimSystem' if hardware == 'gazebo' else 'mock_components/GenericSystem'}"/>
@@ -16,5 +17,7 @@
   <xacro:property name="use_xacro_load_yaml" value="true"/>
   <xacro:property name="mesh_suffix" value="stl"/>
-  <xacro:property name="mesh_path" value="${'file://$(find xarm_description)/meshes' if hardware == 'gazebo' else 'package://xarm_description/meshes'}"/>
+  <!-- UFACTORY's meshes reduced to within 1 mm of their surfaces (scripts/simplify_meshes.py):
+       every camera image and collision check processes them. -->
+  <xacro:property name="mesh_path" value="${'file://$(find arm_description)/meshes/sim' if hardware == 'gazebo' else 'package://arm_description/meshes/sim'}"/>
   <xacro:include filename="$(find arm_description)/urdf/materials.xacro"/>
   <xacro:xarm_materials/>

Commit message: Simulate the wrist D435i's IMU under Bullet Featherstone
gz-physics 9's Bullet Featherstone plugin reports zero velocity for every
non-base link and no link accelerations, so Gazebo's Imu system gave a wrist
IMU only noise and gravity's direction. arm_bringup::PoseImu takes the Imu
system's place for the robot's IMUs. After physics each step it derives
angular velocity from the sensor's rotation over the step and acceleration
from the change in its velocity, averaged over the 10 ms controller period
for which gz_ros2_control holds each velocity command. It low-passes both
like the BMI055 and publishes through gz-sensors' ImuSensor with the SDF
noise. It also removes the sensor's motion components, which Physics would
otherwise query the engine for every step.

WRIST_IMU=true (wrist_imu:=true) adds the D435i IMU at realsense-ros's frame:
/camera/wrist/imu, sensor_msgs/Imu at 200 Hz without orientation, with
BMI055 noise and a per-run turn-on bias (IMU_NOISE=false removes both).

scripts/check_imu.py (make imu-check) sweeps the arm and compares the IMU
with the motion of its frame in TF. With noise, after the biases estimated
at rest, the gyro was within 0.001-0.003 rad/s RMS of a 0.125 rad/s
reference (correlation >= 0.9998), and the wrist's own acceleration
(0.03 m/s^2 RMS) correlated 0.95-0.97. Under DART, whose engine reports link
velocities, the same rotation math matched Gazebo's own gyro to 1e-4 rad/s
RMS. DART's accelerometer misses the accelerations of its velocity servos,
so it was no reference for acceleration.

Two gz-sim behaviours shaped the system:
- Physics implements ConfigurePriority but never registers it with its
  plugin. It therefore runs at the default priority, after any
  kPostPhysicsSensorPriority system, so PoseImu runs at the default + 1.
- Quaternion::AxisAngle takes acos(w), and rounding puts w of a tiny
  per-step rotation just above 1, giving NaN. The angle comes from atan2.

The IMU costs 1-2% of a core in Gazebo (12-20 us of thread CPU per 1 ms
step), against ~7.5% for Gazebo's Imu system plus a system filling in the
motion. The Gazebo, obstacle-course, IMU and mock smoke tests all pass.

Co-Authored-By: Claude Opus 5.5 <noreply@anthropic.com>
Claude-Session: https://claude.ai/code/session_015jsjLXS2XXuwPhcf7UDz3m

File: src/arm_description/urdf/cameras.xacro (robot description, xacro)
@@ -6,4 +6,5 @@
   Gazebo topics  /camera/<name>/color/{image,camera_info}
                  /camera/<name>/depth/{image,camera_info,image/points}
+                 /camera/<name>/imu   (D435i, with wrist_imu)
   frame_id       the optical frame of each imager (z forward, x right, y down)
   Separate sensors rather than one rgbd_camera keep each imager's field of
@@ -55,4 +56,56 @@
         optical_frame="${depth_optical}" width="640" height="360" hfov="1.5184"
         update_rate="${update_rate}" near="0.17" far="10.0" noise="0"/>
+  </xacro:macro>
+  <!-- The D435i's BMI055 IMU, at realsense-ros's frame (_d435i_imu_modules.urdf.xacro,
+       relative to camera_link) and as its unified imu topic at the gyro's
+       200 Hz. Noise follows the BMI055 datasheet (gyro 0.014 deg/s/sqrt(Hz),
+       accel 150 ug/sqrt(Hz)); each run draws a turn-on bias with the
+       datasheet's typical offsets (1 deg/s, 70 mg) as one sigma, as for an
+       uncalibrated unit. The device reports no orientation.
+       Bullet Featherstone reports no link motion to Gazebo's Imu system, so
+       arm_bringup::PoseImu takes its place and measures the motion from the
+       sensor's pose (see pose_imu.cpp). It loads with the robot, so its
+       per-step cost is paid only with the IMU. -->
+  <xacro:macro name="d435i_imu" params="name frame_prefix camera_link update_rate:=200.0 noise:=true">
+    <link name="${frame_prefix}_imu_frame"/>
+    <joint name="${frame_prefix}_imu_joint" type="fixed">
+      <parent link="${camera_link}"/><child link="${frame_prefix}_imu_frame"/>
+      <origin xyz="-0.01174 -0.00552 0.0051" rpy="0 0 0"/>
+    </joint>
+    <link name="${frame_prefix}_imu_optical_frame"/>
+    <joint name="${frame_prefix}_imu_optical_joint" type="fixed">
+      <parent link="${frame_prefix}_imu_frame"/><child link="${frame_prefix}_imu_optical_frame"/>
+      <origin xyz="0 0 0" rpy="${-pi/2} 0 ${-pi/2}"/>
+    </joint>
+    <xacro:macro name="imu_axis_noise" params="stddev bias">
+      <noise type="gaussian"><mean>0</mean><stddev>${stddev if str(noise).lower() == 'true' else 0}</stddev>
+        <bias_mean>0</bias_mean><bias_stddev>${bias if str(noise).lower() == 'true' else 0}</bias_stddev></noise>
+    </xacro:macro>
+    <gazebo reference="${frame_prefix}_imu_optical_frame">
+      <sensor name="${name}_imu" type="imu">
+        <always_on>true</always_on>
+        <update_rate>${update_rate}</update_rate>
+        <topic>/camera/${name}/imu</topic>
+        <gz_frame_id>${frame_prefix}_imu_optical_frame</gz_frame_id>
+        <imu>
+          <enable_orientation>false</enable_orientation>
+          <!-- 0.014 deg/s/sqrt(Hz) over the 100 Hz half-rate band; 1 deg/s bias. -->
+          <angular_velocity>
+            <x><xacro:imu_axis_noise stddev="0.00244" bias="0.01745"/></x>
+            <y><xacro:imu_axis_noise stddev="0.00244" bias="0.01745"/></y>
+            <z><xacro:imu_axis_noise stddev="0.00244" bias="0.01745"/></z>
+          </angular_velocity>
+          <!-- 150 ug/sqrt(Hz) over a 31 Hz band (62.5 Hz accel); 70 mg bias. -->
+          <linear_acceleration>
+            <x><xacro:imu_axis_noise stddev="0.0082" bias="0.687"/></x>
+            <y><xacro:imu_axis_noise stddev="0.0082" bias="0.687"/></y>
+            <z><xacro:imu_axis_noise stddev="0.0082" bias="0.687"/></z>
+          </linear_acceleration>
+        </imu>
+      </sensor>
+    </gazebo>
+    <gazebo>
+      <plugin filename="arm_pose_imu" name="arm_bringup::PoseImu"/>
+    </gazebo>
   </xacro:macro>
   <!-- Intel RealSense D455: color 640x400 at 90 x 65 deg; depth 640x360 at

File: src/arm_description/urdf/xarm6.urdf.xacro (robot description, xacro)
@@ -11,4 +11,6 @@
   <xacro:arg name="camera_hz" default="15.0"/>
   <xacro:arg name="camera_anti_aliasing" default="0"/>
+  <xacro:arg name="wrist_imu" default="false"/>
+  <xacro:arg name="imu_noise" default="true"/>
   <xacro:property name="hardware" value="$(arg hardware)"/>
   <xacro:property name="control_plugin" value="${'gz_ros2_control/GazeboSimSystem' if hardware == 'gazebo' else 'mock_components/GenericSystem'}"/>
@@ -72,4 +74,7 @@
       <xacro:d435i_camera name="wrist" color_link="camera_color_frame" color_optical="camera_color_optical_frame"
           depth_link="camera_depth_frame" depth_optical="camera_depth_optical_frame" update_rate="$(arg camera_hz)"/>
+      <xacro:if value="$(arg wrist_imu)">
+        <xacro:d435i_imu name="wrist" frame_prefix="camera" camera_link="camera_link" noise="$(arg imu_noise)"/>
+      </xacro:if>
     </xacro:if>
   </xacro:if>
